File: KiCAD/CircuitBlockVoltmeter/CircuitBlockVoltmeter.kicad_sch (KiCad schematic)
At the start: 23 parts, among them J1 SSD1306_128x32_OLED, J2 PowerBoost_500C, J3 Conn_01x02_Pin, SW1 SW_SPDT, U1 ATtiny85-20P, U4 OPA2340, U5 LM385BZ-2.5, U6 OPA2340

Commit message: Edit CAD
Parts:
- removed U4, U6: OPA2340, Package_SO:SOIC-8_3.9x4.9mm_P1.27mm, symbol Amplifier_Operational:OPA2340
- added R11: 0, Resistor_THT:R_Axial_DIN0207_L6.3mm_D2.5mm_P7.62mm_Horizontal, symbol Device:R_US
- added U2: OPA4340UA, Package_SO:SOIC-14_3.9x8.7mm_P1.27mm, symbol Amplifier_Operational:OPA4340UA
- J2: footprint (none) -> User:PowerBoost 500C
- R12, R13, R14: footprint Resistor_THT:R_Axial_DIN0207_L6.3mm_D2.5mm_P2.54mm_Vertical -> Resistor_THT:R_Axial_DIN0207_L6.3mm_D2.5mm_P7.62mm_Horizontal
- R4, R5: footprint Resistor_THT:R_Axial_DIN0207_L6.3mm_D2.5mm_P2.54mm_Vertical -> Resistor_THT:R_Axial_DIN0207_L6.3mm_D2.5mm_P10.16mm_Horizontal
- R6: footprint Resistor_THT:R_Axial_DIN0207_L6.3mm_D2.5mm_P5.08mm_Vertical -> Resistor_THT:R_Axial_DIN0207_L6.3mm_D2.5mm_P10.16mm_Horizontal
- R8: footprint Resistor_THT:R_Axial_DIN0207_L6.3mm_D2.5mm_P10.16mm_Horizontal -> Resistor_THT:R_Axial_DIN0207_L6.3mm_D2.5mm_P7.62mm_Horizontal
Connections:
- net +5V: now also J2.1 (5V), U2.4 (V+); no longer J2.5V (Pin_1)
- net AGND: now also U2.1, U2.10 (+), U2.2 (-)
- net AIN: now also U2.8
- net AREF: now also R11.1, R11.2, U2.13 (-), U2.14
- net GND: now also J2.2 (GND), J2.4 (GND), J2.7 (GND), SW1.2 (B), U2.11 (V-); no longer J2.GND (Pin_2), SW1.3 (C)
- net at R5.2, R6.1: now also U2.5 (+)
- net at R1.2, U5.2 (K): now also U2.12 (+)
- net at RV1.2: now also U2.9 (-)
- net at R2.2, R3.1: now also U2.3 (+)
- net at R7.2, R8.2: now also U2.7
- net at R4.2, R7.1: now also U2.6 (-)
- new net: J2.5 (EN), SW1.3 (C)
Other:
- moved on the sheet: R8, SW1
